Commit message: update models
add examples and mvp
change model parameters

File: gripper/urdf/gripper.urdf (robot description, URDF)
Before this commit: robot gripper, 4 links, 3 joints
Links:
- removed link Grip_Base
- removed link Grip_Rotator
- removed link Gripper_1
- removed link Gripper_2
- added link glink1, mass 0.161003401535982; collision mesh filename=package://gripper/meshes/Grip_Rotator.STL; visual mesh filename=package://gripper/meshes/Grip_Rotator.STL
- added link glink2, mass 0.0601996441483964; collision mesh filename=package://gripper/meshes/Gripper_1.STL; visual mesh filename=package://gripper/meshes/Gripper_1.STL
- added link glink3, mass 0.0602; collision mesh filename=package://gripper/meshes/Gripper_2.STL; visual mesh filename=package://gripper/meshes/Gripper_2.STL
- added link gripper_base, mass 1.13983632906086; collision mesh filename=package://gripper/meshes/Grip_Base.STL; visual mesh filename=package://gripper/meshes/Grip_Base.STL
Joints:
- removed joint grip_rot
- removed joint open_1
- removed joint open_2
- added joint gjoint1: type continuous, parent gripper_base, child glink1, origin xyz=0 0 0.10861 rpy=0 0 0, axis 0 0 1, limit effort=0 velocity=0
- added joint gjoint2: type prismatic, parent glink1, child glink2, origin xyz=0 0 0.1071 rpy=0 0 1.5708, axis -1 0 0, limit lower=0 upper=0.064 effort=0 velocity=0
- added joint gjoint3: type prismatic, parent glink1, child glink3, origin xyz=0 0 0.1071 rpy=1.5708 0 -1.5708, axis -1 0 0, limit lower=0 upper=0.064 effort=0 velocity=0

File: robot_arm/urdf/robossembler_arm.urdf (robot description, URDF)
Before this commit: robot rasmt, 8 links, 7 joints
Links:
- removed link Base_Link
- removed link Dock_Link
- removed link Fork_1
- removed link Fork_2
- removed link Fork_3
- removed link Link_1
- removed link Link_2
- removed link Tool_Base
- added link base_link, mass 1.88031044620482; collision mesh filename=package://robot_arm/meshes/Base_Link.stl; visual mesh filename=package://robot_arm/meshes/Base_Link.stl
- added link link1, mass 1.12472202892859; collision mesh filename=package://viewer/meshes/collision/Fork_1.stl; visual mesh filename=package://robot_arm/meshes/Fork_1.stl
- added link link2, mass 1.58688811563124; collision mesh filename=package://viewer/meshes/collision/Link_1.stl; visual mesh filename=package://robot_arm/meshes/Link_1.stl
- added link link3, mass 1.12472202892859; collision mesh filename=package://viewer/meshes/collision/Fork_2.stl; visual mesh filename=package://robot_arm/meshes/Fork_2.stl
- added link link4, mass 1.58688811045173; collision mesh filename=package://viewer/meshes/collision/Link_2.stl; visual mesh filename=package://robot_arm/meshes/Link_2.stl
- added link link5, mass 1.12472202892859; collision mesh filename=package://viewer/meshes/collision/Fork_3.stl; visual mesh filename=package://robot_arm/meshes/Fork_3.stl
- added link link6, mass 1.26942368542312; collision mesh filename=package://viewer/meshes/collision/Dock_Link.stl; visual mesh filename=package://robot_arm/meshes/Dock_Link.stl
- added link tool0
Joints:
- removed joint rot_1
- removed joint rot_2
- removed joint rot_3
- removed joint rot_4
- removed joint rot_5
- removed joint rot_6
- added joint joint1: type revolute, parent base_link, child link1, origin xyz=0 0 0.201360610569537 rpy=0 0 0, axis 0 0 1, limit lower=-3.1416 upper=3.1416 effort=0 velocity=0
- added joint joint2: type revolute, parent link1, child link2, origin xyz=0.11 0 0.115 rpy=0 0 0, axis 0 1 0, limit lower=-1.5708 upper=3.1415 effort=0 velocity=0
- added joint joint3: type revolute, parent link2, child link3, origin xyz=0.001 0 0.156 rpy=0 0 0, axis 0 0 1, limit lower=-3.1416 upper=3.1416 effort=0 velocity=0
- added joint joint4: type revolute, parent link3, child link4, origin xyz=0.11 0 0.115 rpy=0 0 0, axis 0 1 0, limit lower=-1.5708 upper=3.1416 effort=0 velocity=0
- added joint joint5: type revolute, parent link4, child link5, origin xyz=-0.000 0 0.156 rpy=0 0 0, axis 0 0 1, limit lower=-3.1416 upper=3.1416 effort=0 velocity=0
- added joint joint6: type revolute, parent link5, child link6, origin xyz=0.11 0 0.115 rpy=0 0 0, axis 0 1 0, limit lower=-1.5708 upper=3.1416 effort=0 velocity=0
- joint tool: child Tool_Base -> tool0; parent Dock_Link -> link6
